Commit message: update repo

File: src/plane_part/urdf/agv_moving_part.urdf.xacro (robot description, xacro)
@@ -140,5 +140,5 @@
     type="fixed">
     <origin
-      xyz="-0.67 0 -0.015"
+      xyz="-0.67 0 0.075"
       rpy="0 0 0" />
     <parent

File: src/plane_part/urdf/plane_part.urdf.xacro (robot description, xacro)
@@ -377,3 +377,56 @@
     <origin xyz="0.55 0.0 0.06" rpy="0.0 0.0 0.0" />
   </joint>
+  <!-- 地面观察者相机 link -->
+  <link name="observer_camera_link">
+    <visual>
+      <origin xyz="0 0 0" rpy="0 0 0"/>
+      <geometry>
+        <box size="0.05 0.05 0.05"/>
+      </geometry>
+      <material name="blue">
+        <color rgba="0 0 1 1"/>
+      </material>
+    </visual>
+    <collision>
+      <origin xyz="0 0 0" rpy="0 0 0"/>
+      <geometry>
+        <box size="0.05 0.05 0.05"/>
+      </geometry>
+    </collision>
+    <inertial>
+      <origin xyz="0 0 0" rpy="0 0 0"/>
+      <mass value="0.01"/>
+      <inertia ixx="1e-6" ixy="0" ixz="0" iyy="1e-6" iyz="0" izz="1e-6"/>
+    </inertial>
+  </link>
+    <joint name="observer_camera_joint" type="fixed">
+    <parent link="world"/>
+    <child link="observer_camera_link"/>
+    <origin xyz="1.0 -2.0 0.9" rpy="0 0 1.5708"/>
+  </joint>
+  <gazebo reference="observer_camera_link">
+    <sensor type="camera" name="observer_camera_sensor">
+      <camera>
+        <horizontal_fov>1.7</horizontal_fov>
+        <image>
+          <width>1920</width>
+          <height>1080</height>
+          <format>R8G8B8</format>
+        </image>
+        <clip>
+          <near>0.1</near>
+          <far>100</far>
+        </clip>
+      </camera>
+      <always_on>true</always_on>
+      <update_rate>30.0</update_rate>
+      <plugin name="gazebo_ros_camera" filename="libgazebo_ros_camera.so">
+        <robotNamespace>/observer_camera</robotNamespace>
+        <cameraName>observer_y</cameraName>
+        <imageTopicName>image_raw</imageTopicName>
+        <cameraInfoTopicName>camera_info</cameraInfoTopicName>
+        <frameName>observer_camera_link</frameName>
+      </plugin>
+    </sensor>
+  </gazebo>
 </robot>
