Commit message: format files

File: src/plane_part/urdf/agv_moving_part.gazebo.xacro (robot description, xacro)
@@ -10,5 +10,6 @@
         <material>Gazebo/Yellow</material>
     </gazebo>
-    <!--ros control plugin>
+    <!--ros
+    control plugin>
     <gazebo>
         <plugin name="gazebo_ros_control" filename="libgazebo_ros_control.so">
@@ -19,11 +20,11 @@
     </gazebo-->
     <gazebo>
-     <plugin name="base_controller" filename="libgazebo_ros_planar_move.so">
-         <commandTopic>cmd_vel</commandTopic>
-         <odometryTopic>odom</odometryTopic>
-         <odometryFrame>odom</odometryFrame>
-         <odometryRate>20.0</odometryRate>
-         <robotBaseFrame>agv_Link</robotBaseFrame>
-     </plugin>
+        <plugin name="base_controller" filename="libgazebo_ros_planar_move.so">
+            <commandTopic>cmd_vel</commandTopic>
+            <odometryTopic>odom</odometryTopic>
+            <odometryFrame>odom</odometryFrame>
+            <odometryRate>20.0</odometryRate>
+            <robotBaseFrame>agv_Link</robotBaseFrame>
+        </plugin>
     </gazebo>
 </robot>

File: src/plane_part/urdf/agv_moving_part.urdf.xacro (robot description, xacro)
@@ -1,392 +1,394 @@
 <?xml version="1.0" encoding="utf-8"?>
-<!-- This URDF was automatically created by SolidWorks to URDF Exporter! Originally created by Stephen Brawner (brawner@gmail.com)
+<!-- This URDF was automatically created by SolidWorks to URDF Exporter! Originally created by
+Stephen Brawner (brawner@gmail.com)
      Commit Version: 1.6.0-4-g7f85cfe  Build Version: 1.6.7995.38578
      For more information, please see http://wiki.ros.org/sw_urdf_exporter -->
 <robot
-  name="plane_part" xmlns:xacro="http://wiki.ros.org/xacro">
-  <!-- include the xacro files-->
-  <xacro:include filename="$(find plane_part)/urdf/agv_moving_part.gazebo.xacro"/>
-  <xacro:include filename="$(find plane_part)/urdf/materials.xacro"/>
-    <xacro:property name="car_mass" value="20.0"/>
-    <xacro:property name="car_offset" value="0.23"/>
-    <xacro:property name="PI" value="3.1415926536"/>
- <link name="agv_Link">
-     <visual>
-         <geometry>
-             <mesh filename="package://plane_part/meshes/agv2_Link.dae" />
-         </geometry>
-         <material name="green"/>
-         <origin rpy="0.0 0.0 0.0" xyz="0 0 0"/>
-     </visual>
-     <collision>
-         <geometry>
-             <mesh filename="package://plane_part/meshes/agv2_Link.dae" />
-         </geometry>
-         <origin rpy="0.0 0.0 0.0" xyz="0 0 0"/>
-     </collision>
-     <inertial>
-         <mass value="${car_mass}"/>
-         <inertia ixx="${car_mass}" ixy="0.0" ixz="0.0" iyy="${car_mass}" iyz="0.0" izz="${car_mass}" />
-     </inertial>
- </link>
-  <joint
-    name="agv_Joint"
-    type="fixed">
-    <origin
-      xyz="0.0 0.0 0.144"
-      rpy="0 0 0" />
-    <parent
-      link="agv_Link" />
-    <child
-      link="support_Link" />
-    <axis
-      xyz="1 0 0" />
-  </joint>
-  <link
-    name="support_Link">
-    <inertial>
-      <origin
-        xyz="0.071702 1.7942E-05 0.0058498"
-        rpy="0 0 0" />
-      <mass
-        value="91.018" />
-      <inertia
-        ixx="6.4041"
-        ixy="-5.4882E-05"
-        ixz="-3.6045E-06"
-        iyy="6.3339"
-        iyz="-1.8817E-05"
-        izz="12.526" />
-    </inertial>
-    <visual>
-      <origin
-        xyz="0 0 0"
-        rpy="0 0 0" />
-      <geometry>
-        <mesh
-          filename="package://plane_part/meshes/support_Link.dae" />
-      </geometry>
-      <material
-        name="">
-        <color
-          rgba="0 1 0 1" />
-      </material>
-    </visual>
-    <collision>
-      <origin
-        xyz="0 0 0"
-        rpy="0 0 0" />
-      <geometry>
-        <mesh
-          filename="package://plane_part/meshes/support_Link.dae" />
-      </geometry>
-    </collision>
-  </link>
-  <joint
-    name="support_Joint"
-    type="fixed">
-    <origin
-      xyz="0.27 0.0 1.197"
-      rpy="0 0 0" />
-    <parent
-      link="support_Link" />
-    <child
-      link="reference_Link" />
-    <axis
-      xyz="1 0 0" />
-  </joint>
-  <link
-    name="reference_Link">
-    <inertial>
-      <origin
-        xyz="-0.36224 -7.2789E-07 -0.21599"
-        rpy="0 0 0" />
-      <mass
-        value="10.768" />
-      <inertia
-        ixx="0.43054"
-        ixy="-4.8572E-17"
-        ixz="3.0383E-17"
-        iyy="0.17237"
-        iyz="2.6573E-17"
-        izz="0.51657" />
-    </inertial>
-    <visual>
-      <origin
-        xyz="0 0 0"
-        rpy="0 0 0" />
-      <geometry>
-        <mesh
-          filename="package://plane_part/meshes/reference_Link.STL" />
-      </geometry>
-      <material
-        name="">
-        <color
-          rgba="0 1 1 1" />
-      </material>
-    </visual>
-    <collision>
-      <origin
-        xyz="0 0 0"
-        rpy="0 0 0" />
-      <geometry>
-        <mesh
-          filename="package://plane_part/meshes/reference_Link.STL" />
-      </geometry>
-    </collision>
-  </link>
-  <joint
-    name="target1_Joint"
-    type="fixed">
-    <origin
-      xyz="-0.67 0 0.075"
-      rpy="0 0 0" />
-    <parent
-      link="reference_Link" />
-    <child
-      link="image_target1" />
-    <axis
-      xyz="1 0 0" />
-  </joint>
-  <link name="image_target1">
-    <visual>
-      <origin
-        xyz="0 0 0"
-        rpy="0 0 0" />
-      <geometry>
-        <mesh
-          filename="package://plane_part/meshes/aruco_marker.dae" scale="1 5 5"/>
-      </geometry>
-      <material
-        name="">
-        <color
-          rgba="1 1 1 1" />
-      </material>
-    </visual>
-  </link>
-  <joint
-    name="target2_Joint"
-    type="fixed">
-    <origin
-      xyz="-0.67 0.515 -0.015"
-      rpy="0 ${PI/2} 0" />
-    <parent
-      link="reference_Link" />
-    <child
-      link="image_target2" />
-    <axis
-      xyz="1 0 0" />
-  </joint>
-  <link name="image_target2">
-    <visual>
-      <origin
-        xyz="0 0 0"
-        rpy="0 0 0" />
-      <geometry>
-        <cylinder radius="0.01" length="0.002"/>
-      </geometry>
-      <material
-        name="">
-        <color
-          rgba="1 1 1 1" />
-      </material>
-    </visual>
-  </link>
-  <joint
-    name="target3_Joint"
-    type="fixed">
-    <origin
-      xyz="-0.67 -0.515 -0.015"
-      rpy="0 ${PI/2} 0" />
-    <parent
-      link="reference_Link" />
-    <child
-      link="image_target3" />
-    <axis
-      xyz="1 0 0" />
-  </joint>
-  <link name="image_target3">
-    <visual>
-      <origin
-        xyz="0 0 0"
-        rpy="0 0 0" />
-      <geometry>
-        <cylinder radius="0.01" length="0.002"/>
-      </geometry>
-      <material
-        name="">
-        <color
-          rgba="1 1 1 1" />
-      </material>
-    </visual>
-  </link>
-  <joint
-    name="target4_Joint"
-    type="fixed">
-    <origin
-      xyz="-0.67 0 -0.545"
-      rpy="0 ${PI/2} 0" />
-    <parent
-      link="reference_Link" />
-    <child
-      link="image_target4" />
-    <axis
-      xyz="1 0 0" />
-  </joint>
-  <link name="image_target4">
-    <visual>
-      <origin
-        xyz="0 0 0"
-        rpy="0 0 0" />
-      <geometry>
-        <cylinder radius="0.01" length="0.002"/>
-      </geometry>
-      <material
-        name="">
-        <color
-          rgba="1 1 1 1" />
-      </material>
-    </visual>
-  </link>
-  <joint
-    name="target5_Joint"
-    type="fixed">
-    <origin
-      xyz="-0.67 0 0.255"
-      rpy="0 0 0" />
-    <parent
-      link="reference_Link" />
-    <child
-      link="image_target5" />
-    <axis
-      xyz="1 0 0" />
-  </joint>
-  <link name="image_target5">
-    <visual>
-      <origin
-        xyz="0 0 0"
-        rpy="0 0 0" />
-      <geometry>
-        <mesh
-          filename="package://plane_part/meshes/aruco_marker2.dae" />
-      </geometry>
-      <material
-        name="">
-        <color
-          rgba="1 1 1 1" />
-      </material>
-    </visual>
-  </link>
-  <joint
-    name="target6_Joint"
-    type="fixed">
-    <origin
-      xyz="0.0 0.515 -0.045"
-      rpy="0 ${PI/2} 0" />
-    <parent
-      link="reference_Link" />
-    <child
-      link="image_target6" />
-    <axis
-      xyz="1 0 0" />
-  </joint>
-  <link name="image_target6">
-    <visual>
-      <origin
-        xyz="0 0 0"
-        rpy="0 0 0" />
-      <geometry>
-        <cylinder radius="0.01" length="0.002"/>
-      </geometry>
-      <material
-        name="">
-        <color
-          rgba="1 1 1 1" />
-      </material>
-    </visual>
-  </link>
-  <joint
-    name="target7_Joint"
-    type="fixed">
-    <origin
-      xyz="0.0 0.515 -0.515"
-      rpy="0 ${PI/2} 0" />
-    <parent
-      link="reference_Link" />
-    <child
-      link="image_target7" />
-    <axis
-      xyz="1 0 0" />
-  </joint>
-  <link name="image_target7">
-    <visual>
-      <origin
-        xyz="0 0 0"
-        rpy="0 0 0" />
-      <geometry>
-        <cylinder radius="0.01" length="0.002"/>
-      </geometry>
-      <material
-        name="">
-        <color
-          rgba="1 1 1 1" />
-      </material>
-    </visual>
-  </link>
-  <joint
-    name="target8_Joint"
-    type="fixed">
-    <origin
-      xyz="0.0 -0.515 -0.045"
-      rpy="0 ${PI/2} 0" />
-    <parent
-      link="reference_Link" />
-    <child
-      link="image_target8" />
-    <axis
-      xyz="1 0 0" />
-  </joint>
-  <link name="image_target8">
-    <visual>
-      <origin
-        xyz="0 0 0"
-        rpy="0 0 0" />
-      <geometry>
-        <cylinder radius="0.01" length="0.002"/>
-      </geometry>
-      <material
-        name="">
-        <color
-          rgba="1 1 1 1" />
-      </material>
-    </visual>
-  </link>
-  <joint
-    name="target9_Joint"
-    type="fixed">
-    <origin
-      xyz="0.0 -0.515 -0.515"
-      rpy="0 ${PI/2} 0" />
-    <parent
-      link="reference_Link" />
-    <child
-      link="image_target9" />
-    <axis
-      xyz="1 0 0" />
-  </joint>
-  <link name="image_target9">
-    <visual>
-      <origin
-        xyz="0 0 0"
-        rpy="0 0 0" />
-      <geometry>
-        <cylinder radius="0.01" length="0.002"/>
-      </geometry>
-      <material
-        name="">
-        <color
-          rgba="1 1 1 1" />
-      </material>
-    </visual>
-  </link>
+    name="plane_part" xmlns:xacro="http://wiki.ros.org/xacro">
+    <!-- include the xacro files-->
+    <xacro:include filename="$(find plane_part)/urdf/agv_moving_part.gazebo.xacro" />
+    <xacro:include filename="$(find plane_part)/urdf/materials.xacro" />
+    <xacro:property name="car_mass" value="20.0" />
+    <xacro:property name="car_offset" value="0.23" />
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
File: src/plane_part/urdf/materials.xacro (robot description, xacro)
@@ -1,36 +1,36 @@
 <?xml version="1.0"?>
 <robot>
-  <material name="black">
-    <color rgba="0.0 0.0 0.0 1.0"/>
-  </material>
-  <material name="blue">
-    <color rgba="0.0 0.0 0.8 1.0"/>
-  </material>
-  <material name="green">
-    <color rgba="0.0 0.8 0.0 1.0"/>
-  </material>
-  <material name="grey">
-    <color rgba="0.2 0.2 0.2 1.0"/>
-  </material>
-  <material name="orange">
-    <color rgba="${255/255} ${108/255} ${10/255} 1.0"/>
-  </material>
-  <material name="brown">
-    <color rgba="${222/255} ${207/255} ${195/255} 1.0"/>
-  </material>
-  <material name="red">
-    <color rgba="0.8 0.0 0.0 1.0"/>
-  </material>
-  <material name="white">
-    <color rgba="1.0 1.0 1.0 1.0"/>
-  </material>
-  <material name="yellow">
-    <color rgba="1.0 1.0 0.0 1.0"/>
-  </material>
-  <material name="chocolate">
-    <color rgba="${210/255} ${105/255} ${30/255} 1.0"/>
-  </material>
-  <material name="purple">
-    <color rgba="${128/255} 0.0 ${128/255} 1.0"/>
-  </material>
+    <material name="black">
+        <color rgba="0.0 0.0 0.0 1.0" />
+    </material>
+    <material name="blue">
+        <color rgba="0.0 0.0 0.8 1.0" />
+    </material>
+    <material name="green">
+        <color rgba="0.0 0.8 0.0 1.0" />
+    </material>
+    <material name="grey">
+        <color rgba="0.2 0.2 0.2 1.0" />
+    </material>
+    <material name="orange">
+        <color rgba="${255/255} ${108/255} ${10/255} 1.0" />
+    </material>
+    <material name="brown">
+        <color rgba="${222/255} ${207/255} ${195/255} 1.0" />
+    </material>
+    <material name="red">
+        <color rgba="0.8 0.0 0.0 1.0" />
+    </material>
+    <material name="white">
+        <color rgba="1.0 1.0 1.0 1.0" />
+    </material>
+    <material name="yellow">
+        <color rgba="1.0 1.0 0.0 1.0" />
+    </material>
+    <material name="chocolate">
+        <color rgba="${210/255} ${105/255} ${30/255} 1.0" />
+    </material>
+    <material name="purple">
+        <color rgba="${128/255} 0.0 ${128/255} 1.0" />
+    </material>
 </robot>

File: src/plane_part/urdf/plane_part.gazebo.xacro (robot description, xacro)
@@ -13,5 +13,6 @@
         <material>Gazebo/Black</material>
     </gazebo>
-    <!--ros control plugin-->
+    <!--ros
+    control plugin-->
     <gazebo>
         <plugin name="gazebo_ros_control" filename="libgazebo_ros_control.so">
@@ -21,49 +22,49 @@
         </plugin>
     </gazebo>
-  <gazebo reference="xiangji_Link">
-      <sensor type="camera" name="camera1">
-          <update_rate>30.0</update_rate>
-          <camera name="head">
-              <horizontal_fov>0.8</horizontal_fov>
-              <image>
-                  <width>1920</width>
-                  <height>1080</height>
-                  <format>R8G8B8</format>
-              </image>
-              <clip>
-                  <near>0.02</near>
-                  <far>300</far>
-              </clip>
-              <noise>
-                  <type>gaussian</type>
-                  <!-- Noise is sampled independently per pixel on each frame.
+    <gazebo reference="xiangji_Link">
+        <sensor type="camera" name="camera1">
+            <update_rate>30.0</update_rate>
+            <camera name="head">
+                <horizontal_fov>0.8</horizontal_fov>
+                <image>
+                    <width>1920</width>
+                    <height>1080</height>
+                    <format>R8G8B8</format>
+                </image>
+                <clip>
+                    <near>0.02</near>
+                    <far>300</far>
+                </clip>
+                <noise>
+                    <type>gaussian</type>
+                    <!-- Noise is sampled independently per pixel on each frame.
                       That pixel's noise value is added to each of its color
                   channels, which at that point lie in the range [0,1]. -->
-                  <mean>0.0</mean>
-                  <stddev>0.007</stddev>
-              </noise>
-          </camera>
-          <plugin name="camera_controller" filename="libgazebo_ros_camera.so">
-              <alwaysOn>true</alwaysOn>
-              <updateRate>0.0</updateRate>
-              <cameraName>camera1</cameraName>
-              <imageTopicName>image_raw</imageTopicName>
-              <cameraInfoTopicName>camera_info</cameraInfoTopicName>
-              <frameName>camera_link_optical</frameName>
-              <!-- setting hackBaseline to anything but 0.0 will cause a misalignment
+                    <mean>0.0</mean>
+                    <stddev>0.007</stddev>
+                </noise>
+            </camera>
+            <plugin name="camera_controller" filename="libgazebo_ros_camera.so">
+                <alwaysOn>true</alwaysOn>
+                <updateRate>0.0</updateRate>
+                <cameraName>camera1</cameraName>
+                <imageTopicName>image_raw</imageTopicName>
+                <cameraInfoTopicName>camera_info</cameraInfoTopicName>
+                <frameName>camera_link_optical</frameName>
+                <!-- setting hackBaseline to anything but 0.0 will cause a misalignment
                   between the gazebo sensor image and the frame it is supposed to
               be attached to -->
-              <hackBaseline>0.0</hackBaseline>
-              <distortionK1>0.0</distortionK1>
-              <distortionK2>0.0</distortionK2>
-              <distortionK3>0.0</distortionK3>
-              <distortionT1>0.0</distortionT1>
-              <distortionT2>0.0</distortionT2>
-              <CxPrime>0</CxPrime>
-              <Cx>0.0</Cx>
-              <Cy>0.0</Cy>
-              <focalLength>0.0</focalLength>
-          </plugin>
-      </sensor>
-  </gazebo>
+                <hackBaseline>0.0</hackBaseline>
+                <distortionK1>0.0</distortionK1>
+                <distortionK2>0.0</distortionK2>
+                <distortionK3>0.0</distortionK3>
+                <distortionT1>0.0</distortionT1>
+                <distortionT2>0.0</distortionT2>
+                <CxPrime>0</CxPrime>
+                <Cx>0.0</Cx>
+                <Cy>0.0</Cy>
+                <focalLength>0.0</focalLength>
+            </plugin>
+        </sensor>
+    </gazebo>
 </robot>

File: src/plane_part/urdf/plane_part.transmission.xacro (robot description, xacro)
@@ -55,5 +55,6 @@
         </actuator>
     </transmission>
-    <!--transmission name="refer01">
+    <!--transmission
+    name="refer01">
         <type>transmission_interface/SimpleTransmission</type>
         <joint name="reference_Joint">
@@ -64,5 +65,6 @@
         </actuator>
     </transmission-->
-    <!--transmission name="trans04_3">
+    <!--transmission
+    name="trans04_3">
         <type>transmission_interface/SimpleTransmission</type>
         <joint name="clap_roll_joint">
