Commit message: format files

File: src/plane_part/urdf/plane_part.urdf.xacro (robot description, xacro)
@@ -1,432 +1,434 @@
 <?xml version="1.0" encoding="utf-8"?>
-<!-- This URDF was automatically created by SolidWorks to URDF Exporter! Originally created by Stephen Brawner (brawner@gmail.com)
+<!-- This URDF was automatically created by SolidWorks to URDF Exporter! Originally created by
+Stephen Brawner (brawner@gmail.com)
      Commit Version: 1.6.0-4-g7f85cfe  Build Version: 1.6.7995.38578
      For more information, please see http://wiki.ros.org/sw_urdf_exporter -->
 <robot
-  name="plane_part" xmlns:xacro="http://wiki.ros.org/xacro">
-  <!-- include the xacro files-->
-  <xacro:include filename="$(find plane_part)/urdf/plane_part.transmission.xacro"/>
-  <xacro:include filename="$(find plane_part)/urdf/plane_part.gazebo.xacro"/>
-  <xacro:include filename="$(find plane_part)/urdf/materials.xacro"/>
-  <xacro:property name="PI" value="3.1415926535897931" />
-  <xacro:macro name="cylinder_inertial" params="radius length mass *origin">
-    <inertial>
-      <mass value="${mass}" />
-      <xacro:insert_block name="origin" />
-      <inertia ixx="${0.0833333 * mass * (3 * radius * radius + length * length)}" ixy="0.0" ixz="0.0"
-        iyy="${0.0833333 * mass * (3 * radius * radius + length * length)}" iyz="0.0"
-        izz="${0.5 * mass * radius * radius}" />
-    </inertial>
-  </xacro:macro>
-  <link name="world"/>
-  <link
-    name="base_link">
-    <inertial>
-      <origin
-        xyz="0.00014734 -0.0013249 -0.027719"
-        rpy="0 0 0" />
-      <mass
-        value="0.90493" />
-      <inertia
-        ixx="0.0011428"
-        ixy="-1.8056E-35"
-        ixz="-1.8016E-20"
-        iyy="0.0011428"
-        iyz="1.7948E-20"
-        izz="0.00050332" />
-    </inertial>
-    <visual>
-      <origin
-        xyz="0 0 0"
-        rpy="0 0 0" />
-      <geometry>
-        <mesh
-          filename="package://plane_part/meshes/base_link.STL" />
-      </geometry>
-      <material
-        name="">
-        <color
-          rgba="1 0 0 1" />
-      </material>
-    </visual>
-    <collision>
-      <origin
-        xyz="0 0 0"
-        rpy="0 0 0" />
-      <geometry>
-        <mesh
-          filename="package://plane_part/meshes/base_link.STL" />
-      </geometry>
-    </collision>
-  </link>
-  <joint name="world_base" type="fixed">
-    <origin rpy="0.0 0.0 0.0" xyz="0.0 0.0 0.1"/>
-    <parent link="world"/>
-    <child link="base_link"/>
-  </joint>
-  <link
-    name="bottom_Link">
-    <inertial>
-      <origin
-        xyz="0.071702 1.7942E-05 0.0058498"
-        rpy="0 0 0" />
-      <mass
-        value="91.018" />
-      <inertia
-        ixx="6.4041"
-        ixy="-5.4882E-05"
-        ixz="-3.6045E-06"
-        iyy="6.3339"
-        iyz="-1.8817E-05"
-        izz="12.526" />
-    </inertial>
-    <visual>
-      <origin
-        xyz="0 0 0"
-        rpy="0 0 0" />
-      <geometry>
-        <mesh
-          filename="package://plane_part/meshes/bottom_Link.dae" />
-      </geometry>
-      <material
-        name="">
-        <color
-          rgba="0 1 0 1" />
-      </material>
-    </visual>
-    <collision>
-      <origin
-        xyz="0 0 0"
-        rpy="0 0 0" />
-      <geometry>
-        <mesh
-          filename="package://plane_part/meshes/bottom_Link.dae" />
-      </geometry>
-    </collision>
-  </link>
-  <joint
-    name="bottom_joint"
-    type="fixed">
-    <origin
-      xyz="0 0 0"
-      rpy="0 0 0" />
-    <parent
-      link="base_link" />
-    <child
-      link="bottom_Link" />
-    <axis
-      xyz="1 0 0" />
-  </joint>
-  <link name="platform_x_Link">
-    <inertial>
-      <origin rpy="0.0 0.0 0.0" xyz="0.0 0.0 0.0"/>
-      <mass value="1"/>
-      <inertia ixx="1" ixy="0.0" ixz="0.0" iyy="1" iyz="0.0" izz="1"/>
-    </inertial>
-  </link>
-  <joint
-    name="platform_x_joint"
-    type="prismatic">
-    <origin
-      xyz="0 0 0.61449"
-      rpy="0 0 0" />
-    <parent
-      link="bottom_Link" />
-    <child
-      link="platform_x_Link" />
-    <axis
-      xyz="1 0 0" />
-    <limit
-      lower="-0.3"
-      upper="0.3"
-      effort="10000.0"
-      velocity="0.1" />
-  </joint>
-  <link name="platform_y_Link">
-    <inertial>
-      <origin rpy="0.0 0.0 0.0" xyz="0.0 0.0 0.0"/>
-      <mass value="1"/>
-      <inertia ixx="1" ixy="0.0" ixz="0.0" iyy="1" iyz="0.0" izz="1"/>
-    </inertial>
-  </link>
-  <joint
-    name="platform_y_joint"
-    type="prismatic">
-    <origin
-      xyz="0 0 0"
-      rpy="0 0 0" />
-    <parent
-      link="platform_x_Link" />
-    <child
-      link="platform_y_Link" />
-    <axis
-      xyz="0 1 0" />
-    <limit
-      lower="-0.3"
-      upper="0.3"
-      effort="10000.0"
-      velocity="0.1" />
-  </joint>
-  <link name="platform_z_Link">
-    <inertial>
-      <origin rpy="0.0 0.0 0.0" xyz="0.0 0.0 0.0"/>
-      <mass value="1"/>
-      <inertia ixx="1" ixy="0.0" ixz="0.0" iyy="1" iyz="0.0" izz="1"/>
-    </inertial>
-  </link>
-  <joint
-    name="platform_z_joint"
-    type="prismatic">
-    <origin
-      xyz="0 0 0"
-      rpy="0 0 0" />
-    <parent
-      link="platform_y_Link" />
-    <child
-      link="platform_z_Link" />
-    <axis
-      xyz="0 0 1" />
-    <limit
-      lower="-0.3"
-      upper="0.3"
-      effort="10000.0"
-      velocity="0.1" />
-  </joint>
-  <link name="platform_a_Link">
-    <inertial>
-      <origin rpy="0.0 0.0 0.0" xyz="0.0 0.0 0.0"/>
-      <mass value="1"/>
-      <inertia ixx="1" ixy="0.0" ixz="0.0" iyy="1" iyz="0.0" izz="1"/>
-    </inertial>
-  </link>
-  <joint
-    name="platform_a_joint"
-    type="revolute">
-    <origin
-      xyz="0 0 0"
-      rpy="0 0 0" />
-    <parent
-      link="platform_z_Link" />
-    <child
-      link="platform_a_Link" />
-    <axis
-      xyz="1 0 0" />
-    <limit
-      lower="-0.3"
-      upper="0.3"
-      effort="10000.0"
-      velocity="0.1" />
-  </joint>
-  <link name="platform_b_Link">
-    <inertial>
-      <origin rpy="0.0 0.0 0.0" xyz="0.0 0.0 0.0"/>
-      <mass value="1"/>
-      <inertia ixx="1" ixy="0.0" ixz="0.0" iyy="1" iyz="0.0" izz="1"/>
-    </inertial>
-  </link>
-  <joint
-    name="platform_b_joint"
-    type="revolute">
-    <origin
-      xyz="0 0 0"
-      rpy="0 0 0" />
-    <parent
-      link="platform_a_Link" />
-    <child
-      link="platform_b_Link" />
-    <axis
-      xyz="0 1 0" />
-    <limit
-      lower="-0.3"
-      upper="0.3"
-      effort="10000.0"
-      velocity="0.1" />
-  </joint>
-  <link
-    name="platform_Link">
-    <inertial>
-      <origin
-        xyz="0.0016018 0.0014397 -0.0097437"
-        rpy="0 0 0" />
-      <mass
-        value="4.3742" />
-      <inertia
-        ixx="0.095075"
-        ixy="-2.0348E-11"
-        ixz="6.0005E-11"
-        iyy="0.094958"
-        iyz="1.164E-11"
-        izz="0.18974" />
-    </inertial>
-    <visual>
-      <origin
-        xyz="0 0 0"
-        rpy="0 0 0" />
-      <geometry>
-        <mesh
-          filename="package://plane_part/meshes/platform_Link.STL" />
-      </geometry>
-      <material
-        name="">
-        <color
-          rgba="0 0 1 1" />
-      </material>
-    </visual>
-    <collision>
-      <origin
-        xyz="0 0 0"
-        rpy="0 0 0" />
-      <geometry>
-        <mesh
-          filename="package://plane_part/meshes/platform_Link.STL" />
-      </geometry>
-    </collision>
-  </link>
-  <joint
-    name="platform_c_Joint"
-    type="revolute">
-    <origin
-      xyz="0 0 0"
-      rpy="0 0 0" />
-    <parent
-      link="platform_b_Link" />
-    <child
-      link="platform_Link" />
-    <axis
-      xyz="0 0 1" />
-    <limit
-      lower="-0.3"
-      upper="0.3"
-      effort="10000.0"
-      velocity="0.1" />
-  </joint>
-  <link
-    name="modulating_Link">
-    <inertial>
-      <origin
-        xyz="0.46708 -6.9672E-07 -0.18298"
-        rpy="0 0 0" />
-      <mass
-        value="11.25" />
-      <inertia
-        ixx="0.40589"
-        ixy="1.2212E-15"
-        ixz="1.6631E-13"
-        iyy="0.28426"
-        iyz="1.2524E-15"
-        izz="0.50773" />
-    </inertial>
-    <visual>
-      <origin
-        xyz="0 0 0"
-        rpy="0 0 0" />
-      <geometry>
-        <mesh
-          filename="package://plane_part/meshes/modulating_Link.STL" />
-      </geometry>
-      <material
-        name="">
-        <color
-          rgba="1 1 0 1" />
-      </material>
-    </visual>
-    <collision>
-      <origin
-        xyz="0 0 0"
-        rpy="0 0 0" />
-      <geometry>
-        <mesh
-          filename="package://plane_part/meshes/modulating_Link.STL" />
-      </geometry>
-    </collision>
-  </link>
-  <joint
-    name="modulating_Joint"
-    type="fixed">
-    <origin
-      xyz="-0.236 0 0.56"
-      rpy="0 0 0" />
-    <parent
-      link="platform_Link" />
-    <child
-      link="modulating_Link" />
-    <axis
-      xyz="1 0 0" />
-  </joint>
-  <link name="xiangji_Link">
-    <visual>
-        <origin xyz="-0.1 0.0 0.0" rpy="0 ${PI/2.0} 0" />
-      <geometry>
-        <mesh filename="package://plane_part/meshes/xiangji.STL"/>
-      </geometry>
-      <material name="orange"/>
-    </visual>
-    <collision>
-        <origin xyz="-0.1 0.0 0.0" rpy="0 ${PI/2.0} 0" />
-      <geometry>
-        <mesh filename="package://plane_part/meshes/xiangji.STL"/>
-      </geometry>
-    </collision>
-    <xacro:cylinder_inertial radius="0.01" length="0.05" mass="0.01">
-      <origin xyz="0.0 0.0 0.0" rpy="0 0 0" />
-    </xacro:cylinder_inertial>
-  </link>
-  <joint name="xiangji_Joint" type="fixed">
-    <parent link="modulating_Link" />
-    <child link = "xiangji_Link" />
-    <origin xyz="0.55 0.0 0.06" rpy="0.0 0.0 0.0" />
-  </joint>
-  <!-- 地面观察者相机 link -->
-  <link name="observer_camera_link">
-    <visual>
-      <origin xyz="0 0 0" rpy="0 0 0"/>
-      <geometry>
-        <box size="0.05 0.05 0.05"/>
-      </geometry>
-      <material name="blue">
-        <color rgba="0 0 1 1"/>
-      </material>
-    </visual>
-    <collision>
-      <origin xyz="0 0 0" rpy="0 0 0"/>
-      <geometry>
-        <box size="0.05 0.05 0.05"/>
-      </geometry>
-    </collision>
-    <inertial>
-      <origin xyz="0 0 0" rpy="0 0 0"/>
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
File: src/plane_part/urdf/plane_part2.urdf.xacro (robot description, xacro)
@@ -1,399 +1,400 @@
 <?xml version="1.0" encoding="utf-8"?>
-<!-- This URDF was automatically created by SolidWorks to URDF Exporter! Originally created by Stephen Brawner (brawner@gmail.com)
+<!-- This URDF was automatically created by SolidWorks to URDF Exporter! Originally created by
+Stephen Brawner (brawner@gmail.com)
      Commit Version: 1.6.0-4-g7f85cfe  Build Version: 1.6.7995.38578
      For more information, please see http://wiki.ros.org/sw_urdf_exporter -->
 <robot
-  name="plane_part" xmlns:xacro="http://wiki.ros.org/xacro">
-  <!-- include the xacro files-->
-  <xacro:include filename="$(find plane_part)/urdf/plane_part.transmission.xacro"/>
-  <xacro:include filename="$(find plane_part)/urdf/plane_part.gazebo.xacro"/>
-  <xacro:include filename="$(find plane_part)/urdf/materials.xacro"/>
-  <link name="world"/>
-  <link
-    name="base_link">
-    <inertial>
-      <origin
-        xyz="0.00014734 -0.0013249 -0.027719"
-        rpy="0 0 0" />
-      <mass
-        value="0.90493" />
-      <inertia
-        ixx="0.0011428"
-        ixy="-1.8056E-35"
-        ixz="-1.8016E-20"
-        iyy="0.0011428"
-        iyz="1.7948E-20"
-        izz="0.00050332" />
-    </inertial>
-    <visual>
-      <origin
-        xyz="0 0 0"
-        rpy="0 0 0" />
-      <geometry>
-        <mesh
-          filename="package://plane_part/meshes/base_link.STL" />
-      </geometry>
-      <material
-        name="">
-        <color
-          rgba="1 0 0 1" />
-      </material>
-    </visual>
-    <collision>
-      <origin
-        xyz="0 0 0"
-        rpy="0 0 0" />
-      <geometry>
-        <mesh
-          filename="package://plane_part/meshes/base_link.STL" />
-      </geometry>
-    </collision>
-  </link>
-  <joint name="world_base" type="fixed">
-    <origin rpy="0.0 0.0 0.0" xyz="0.0 0.0 0.2"/>
-    <parent link="world"/>
-    <child link="base_link"/>
-  </joint>
-  <link
-    name="bottom_Link">
-    <inertial>
-      <origin
-        xyz="0.071702 1.7942E-05 0.0058498"
-        rpy="0 0 0" />
-      <mass
-        value="91.018" />
-      <inertia
-        ixx="6.4041"
-        ixy="-5.4882E-05"
-        ixz="-3.6045E-06"
-        iyy="6.3339"
-        iyz="-1.8817E-05"
-        izz="12.526" />
-    </inertial>
-    <visual>
-      <origin
-        xyz="0 0 0"
-        rpy="0 0 0" />
-      <geometry>
-        <mesh
-          filename="package://plane_part/meshes/bottom_Link.STL" />
-      </geometry>
-      <material
-        name="">
-        <color
-          rgba="0 1 0 1" />
-      </material>
-    </visual>
-    <collision>
-      <origin
-        xyz="0 0 0"
-        rpy="0 0 0" />
-      <geometry>
-        <mesh
-          filename="package://plane_part/meshes/bottom_Link.STL" />
-      </geometry>
-    </collision>
-  </link>
-  <joint
-    name="bottom_joint"
-    type="fixed">
-    <origin
-      xyz="0 0 0"
-      rpy="0 0 0" />
-    <parent
-      link="base_link" />
-    <child
-      link="bottom_Link" />
-    <axis
-      xyz="1 0 0" />
-  </joint>
-  <link name="platform_x_Link">
-    <inertial>
-      <origin rpy="0.0 0.0 0.0" xyz="0.0 0.0 0.0"/>
-      <mass value="1"/>
-      <inertia ixx="1" ixy="0.0" ixz="0.0" iyy="1" iyz="0.0" izz="1"/>
-    </inertial>
-  </link>
-  <joint
-    name="platform_x_joint"
-    type="prismatic">
-    <origin
-      xyz="0 0 0.61449"
-      rpy="0 0 0" />
-    <parent
-      link="bottom_Link" />
-    <child
-      link="platform_x_Link" />
-    <axis
-      xyz="1 0 0" />
-    <limit
-      lower="-0.3"
-      upper="0.3"
-      effort="10000.0"
-      velocity="0.1" />
-  </joint>
-  <link name="platform_y_Link">
-    <inertial>
-      <origin rpy="0.0 0.0 0.0" xyz="0.0 0.0 0.0"/>
-      <mass value="1"/>
-      <inertia ixx="1" ixy="0.0" ixz="0.0" iyy="1" iyz="0.0" izz="1"/>
-    </inertial>
-  </link>
-  <joint
-    name="platform_y_joint"
-    type="prismatic">
-    <origin
-      xyz="0 0 0"
-      rpy="0 0 0" />
-    <parent
-      link="platform_x_Link" />
-    <child
-      link="platform_y_Link" />
-    <axis
-      xyz="0 1 0" />
-    <limit
-      lower="-0.3"
-      upper="0.3"
-      effort="10000.0"
-      velocity="0.1" />
-  </joint>
-  <link name="platform_z_Link">
-    <inertial>
-      <origin rpy="0.0 0.0 0.0" xyz="0.0 0.0 0.0"/>
-      <mass value="1"/>
-      <inertia ixx="1" ixy="0.0" ixz="0.0" iyy="1" iyz="0.0" izz="1"/>
-    </inertial>
-  </link>
-  <joint
-    name="platform_z_joint"
-    type="prismatic">
-    <origin
-      xyz="0 0 0"
-      rpy="0 0 0" />
-    <parent
-      link="platform_y_Link" />
-    <child
-      link="platform_z_Link" />
-    <axis
-      xyz="0 0 1" />
-    <limit
-      lower="-0.3"
-      upper="0.3"
-      effort="10000.0"
-      velocity="0.1" />
-  </joint>
-  <link name="platform_a_Link">
-    <inertial>
-      <origin rpy="0.0 0.0 0.0" xyz="0.0 0.0 0.0"/>
-      <mass value="1"/>
-      <inertia ixx="1" ixy="0.0" ixz="0.0" iyy="1" iyz="0.0" izz="1"/>
-    </inertial>
-  </link>
-  <joint
-    name="platform_a_joint"
-    type="revolute">
-    <origin
-      xyz="0 0 0"
-      rpy="0 0 0" />
-    <parent
-      link="platform_z_Link" />
-    <child
-      link="platform_a_Link" />
-    <axis
-      xyz="1 0 0" />
-    <limit
-      lower="-0.3"
-      upper="0.3"
-      effort="10000.0"
-      velocity="0.1" />
-  </joint>
-  <link name="platform_b_Link">
-    <inertial>
-      <origin rpy="0.0 0.0 0.0" xyz="0.0 0.0 0.0"/>
-      <mass value="1"/>
-      <inertia ixx="1" ixy="0.0" ixz="0.0" iyy="1" iyz="0.0" izz="1"/>
-    </inertial>
-  </link>
-  <joint
-    name="platform_b_joint"
-    type="revolute">
-    <origin
-      xyz="0 0 0"
-      rpy="0 0 0" />
-    <parent
-      link="platform_a_Link" />
-    <child
-      link="platform_b_Link" />
-    <axis
-      xyz="0 1 0" />
-    <limit
-      lower="-0.3"
-      upper="0.3"
-      effort="10000.0"
-      velocity="0.1" />
-  </joint>
-  <link
-    name="platform_Link">
-    <inertial>
-      <origin
-        xyz="0.0016018 0.0014397 -0.0097437"
-        rpy="0 0 0" />
-      <mass
-        value="4.3742" />
-      <inertia
-        ixx="0.095075"
-        ixy="-2.0348E-11"
-        ixz="6.0005E-11"
-        iyy="0.094958"
-        iyz="1.164E-11"
-        izz="0.18974" />
-    </inertial>
-    <visual>
-      <origin
-        xyz="0 0 0"
-        rpy="0 0 0" />
-      <geometry>
-        <mesh
-          filename="package://plane_part/meshes/platform_Link.STL" />
-      </geometry>
-      <material
-        name="">
-        <color
-          rgba="0 0 1 1" />
-      </material>
-    </visual>
-    <collision>
-      <origin
-        xyz="0 0 0"
-        rpy="0 0 0" />
-      <geometry>
-        <mesh
-          filename="package://plane_part/meshes/platform_Link.STL" />
-      </geometry>
-    </collision>
-  </link>
-  <joint
-    name="platform_c_Joint"
-    type="revolute">
-    <origin
-      xyz="0 0 0"
-      rpy="0 0 0" />
-    <parent
-      link="platform_b_Link" />
-    <child
-      link="platform_Link" />
-    <axis
-      xyz="0 0 1" />
-    <limit
-      lower="-0.3"
-      upper="0.3"
-      effort="10000.0"
-      velocity="0.1" />
-  </joint>
-  <link
-    name="modulating_Link">
-    <inertial>
-      <origin
-        xyz="0.46708 -6.9672E-07 -0.18298"
-        rpy="0 0 0" />
-      <mass
-        value="11.25" />
-      <inertia
-        ixx="0.40589"
-        ixy="1.2212E-15"
-        ixz="1.6631E-13"
-        iyy="0.28426"
-        iyz="1.2524E-15"
-        izz="0.50773" />
-    </inertial>
-    <visual>
-      <origin
-        xyz="0 0 0"
-        rpy="0 0 0" />
-      <geometry>
-        <mesh
-          filename="package://plane_part/meshes/modulating_Link.STL" />
-      </geometry>
-      <material
-        name="">
-        <color
-          rgba="1 1 0 1" />
-      </material>
-    </visual>
-    <collision>
-      <origin
-        xyz="0 0 0"
-        rpy="0 0 0" />
-      <geometry>
-        <mesh
-          filename="package://plane_part/meshes/modulating_Link.STL" />
-      </geometry>
-    </collision>
-  </link>
-  <joint
-    name="modulating_Joint"
-    type="fixed">
-    <origin
-      xyz="-0.2495352 -0.0100989 0.5408577"
-      rpy="-0.0099 0.0049 -0.0113" />
-    <parent
-      link="platform_Link" />
-    <child
-      link="modulating_Link" />
-    <axis
-      xyz="1 0 0" />
-  </joint>
-  <link
-    name="reference_Link">
-    <inertial>
-      <origin
-        xyz="-0.36224 -7.2789E-07 -0.21599"
-        rpy="0 0 0" />
-      <mass
-        value="10.768" />
-      <inertia
-        ixx="0.43054"
-        ixy="-4.8572E-17"
-        ixz="3.0383E-17"
-        iyy="0.17237"
-        iyz="2.6573E-17"
-        izz="0.51657" />
-    </inertial>
-    <visual>
-      <origin
-        xyz="0 0 0"
-        rpy="0 0 0" />
-      <geometry>
-        <mesh
-          filename="package://plane_part/meshes/reference_Link.STL" />
-      </geometry>
-      <material
-        name="">
-        <color
-          rgba="0 1 1 1" />
-      </material>
-    </visual>
-    <collision>
-      <origin
-        xyz="0 0 0"
-        rpy="0 0 0" />
-      <geometry>
-        <mesh
-          filename="package://plane_part/meshes/reference_Link.STL" />
-      </geometry>
-    </collision>
-  </link>
-  <joint
-    name="reference_Joint"
-    type="fixed">
-    <origin
-      xyz="1.3264 -0.0925 1.1924"
-      rpy="-0.0047 0.007 -0.0023" />
-    <parent
-      link="bottom_Link" />
-    <child
-      link="reference_Link" />
-    <axis
-      xyz="1 0 0" />
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